Commit message: Link 5: head box end wall 3 mm clear of the forearm tube (was tangent - zero-length edges, no FE mesh); URDF, dynamics and strength data regenerated
Co-Authored-By: Claude Opus 5.5 <noreply@anthropic.com>
Claude-Session: https://claude.ai/code/session_01HNc2e7dHna5JzqoB2AUz2M

File: sim/RTC-7/RTC-7.urdf (robot description, URDF)
Before this commit: robot RTC7, 10 links, 9 joints
Links:
- link link_5: mass 10.7250 -> 10.7593
